Commit message: Update irb2600_12_165.urdf

File: abb_irb2600_support/urdf/irb2600_12_165.urdf (robot description, URDF)
Before this commit: robot abb_irb2600_12_165, 10 links, 9 joints
Links:
- link base_link: geometry collision mesh filename=package://abb_irb2600_support/meshes/collision/base_link.stl; visual mesh filename=package://abb_irb2600_support/meshes/visual/base_link.stl
- link link_1: geometry collision mesh filename=package://abb_irb2600_support/meshes/collision/link_1.stl; visual mesh filename=package://abb_irb2600_support/meshes/visual/link_1.stl
- link link_2: geometry collision mesh filename=package://abb_irb2600_support/meshes/collision/link_2.stl; visual mesh filename=package://abb_irb2600_support/meshes/visual/link_2.stl
- link link_3: geometry collision mesh filename=package://abb_irb2600_support/meshes/collision/link_3.stl; visual mesh filename=package://abb_irb2600_support/meshes/visual/link_3.stl
- link link_4: geometry collision mesh filename=package://abb_irb2600_support/meshes/collision/link_4.stl; visual mesh filename=package://abb_irb2600_support/meshes/visual/link_4.stl
- link link_5: geometry collision mesh filename=package://abb_irb2600_support/meshes/collision/link_5.stl; visual mesh filename=package://abb_irb2600_support/meshes/visual/link_5.stl
- link link_6: geometry collision mesh filename=package://abb_irb2600_support/meshes/collision/link_6.stl; visual mesh filename=package://abb_irb2600_support/meshes/visual/link_6.stl
